Commit message: feat: add control and sensor configurations

File: src/vineyard_mower_description/urdf/vineyard_mower.urdf.xacro (robot description, xacro)
@@ -274,18 +274,167 @@
     <material>Gazebo/Blue</material>
   </gazebo>
-  <!-- Differential drive plugin for Gz -->
+  <!-- ros2_control -->
+  <ros2_control name="GazeboSystem" type="system">
+    <hardware>
+      <plugin>gz_ros2_control/GazeboSimSystem</plugin>
+    </hardware>
+    <joint name="left_wheel_joint">
+      <command_interface name="velocity">
+        <param name="min">-10</param>
+        <param name="max">10</param>
+      </command_interface>
+      <state_interface name="velocity"/>
+      <state_interface name="position"/>
+    </joint>
+    <joint name="right_wheel_joint">
+      <command_interface name="velocity">
+        <param name="min">-10</param>
+        <param name="max">10</param>
+      </command_interface>
+      <state_interface name="velocity"/>
+      <state_interface name="position"/>
+    </joint>
+  </ros2_control>
+  <!-- Gazebo ros2_control plugin -->
   <gazebo>
-    <plugin filename="gz-sim-diff-drive-system" name="gz::sim::systems::DiffDrive">
-      <left_joint>left_wheel_joint</left_joint>
-      <right_joint>right_wheel_joint</right_joint>
-      <wheel_separation>${track_width}</wheel_separation>
-      <wheel_radius>${wheel_radius}</wheel_radius>
-      <odom_publish_frequency>1</odom_publish_frequency>
-      <topic>cmd_vel</topic>
-      <odom_topic>odom</odom_topic>
-      <tf_topic>/tf</tf_topic>
-      <frame_id>odom</frame_id>
-      <child_frame_id>base_link</child_frame_id>
+    <plugin filename="gz_ros2_control-system" name="gz_ros2_control::GazeboSimROS2ControlPlugin">
+      <parameters>$(find vineyard_mower_description)/config/control_config.yaml</parameters>
     </plugin>
   </gazebo>
+  <!-- LiDAR sensor plugin -->
+  <gazebo reference="lidar_link">
+    <sensor name="lidar" type="gpu_lidar">
+      <topic>scan</topic>
+      <update_rate>10</update_rate>
+      <lidar>
+        <scan>
+          <horizontal>
+            <samples>360</samples>
+            <resolution>1</resolution>
+            <min_angle>-3.141592</min_angle>
+            <max_angle>3.141592</max_angle>
+          </horizontal>
+          <vertical>
+            <samples>1</samples>
+            <resolution>1</resolution>
+            <min_angle>0</min_angle>
+            <max_angle>0</max_angle>
+          </vertical>
+        </scan>
+        <range>
+          <min>0.1</min>
+          <max>30.0</max>
+          <resolution>0.01</resolution>
+        </range>
+      </lidar>
+      <always_on>1</always_on>
+      <visualize>true</visualize>
+    </sensor>
+  </gazebo>
+  <!-- Front camera sensor plugin (Intel RealSense simulation) -->
+  <gazebo reference="front_camera_link">
+    <sensor name="front_camera" type="rgbd_camera">
+      <topic>front_camera</topic>
+      <update_rate>30</update_rate>
+      <camera>
+        <horizontal_fov>1.047198</horizontal_fov>
+        <image>
+          <width>640</width>
+          <height>480</height>
+          <format>R8G8B8</format>
+        </image>
+        <clip>
+          <near>0.1</near>
+          <far>10.0</far>
+        </clip>
+      </camera>
+      <always_on>1</always_on>
+      <visualize>true</visualize>
+    </sensor>
+  </gazebo>
+  <!-- Rear camera sensor plugin (Intel RealSense simulation) -->
+  <gazebo reference="rear_camera_link">
+    <sensor name="rear_camera" type="rgbd_camera">
+      <topic>rear_camera</topic>
+      <update_rate>30</update_rate>
+      <camera>
+        <horizontal_fov>1.047198</horizontal_fov>
+        <image>
+          <width>640</width>
+          <height>480</height>
+          <format>R8G8B8</format>
+        </image>
+        <clip>
+          <near>0.1</near>
+          <far>10.0</far>
+        </clip>
+      </camera>
+      <always_on>1</always_on>
+      <visualize>true</visualize>
+    </sensor>
+  </gazebo>
+  <!-- IMU sensor for additional odometry -->
+  <link name="imu_link">
+    <inertial>
+      <origin xyz="0 0 0" rpy="0 0 0"/>
+      <mass value="0.1"/>
+      <inertia ixx="0.001" ixy="0" ixz="0" iyy="0.001" iyz="0" izz="0.001"/>
+    </inertial>
+  </link>
+  <joint name="imu_joint" type="fixed">
+    <parent link="upper_chassis"/>
+    <child link="imu_link"/>
+    <origin xyz="0 0 0" rpy="0 0 0"/>
+  </joint>
+  <!-- IMU sensor plugin -->
+  <gazebo reference="imu_link">
+    <sensor name="imu_sensor" type="imu">
+      <topic>imu</topic>
+      <update_rate>100</update_rate>
+      <imu>
+        <angular_velocity>
+          <x>
+            <noise type="gaussian">
+              <mean>0.0</mean>
+              <stddev>2e-4</stddev>
+            </noise>
+          </x>
+          <y>
+            <noise type="gaussian">
+              <mean>0.0</mean>
+              <stddev>2e-4</stddev>
+            </noise>
+          </y>
+          <z>
+            <noise type="gaussian">
+              <mean>0.0</mean>
+              <stddev>2e-4</stddev>
+            </noise>
+          </z>
+        </angular_velocity>
+        <linear_acceleration>
+          <x>
+            <noise type="gaussian">
+              <mean>0.0</mean>
+              <stddev>1.7e-2</stddev>
+            </noise>
+          </x>
+          <y>
+            <noise type="gaussian">
+              <mean>0.0</mean>
+              <stddev>1.7e-2</stddev>
+            </noise>
+          </y>
+          <z>
+            <noise type="gaussian">
+              <mean>0.0</mean>
+              <stddev>1.7e-2</stddev>
+            </noise>
+          </z>
+        </linear_acceleration>
+      </imu>
+      <always_on>1</always_on>
+      <visualize>true</visualize>
+    </sensor>
+  </gazebo>
 </robot>

Commit message: fix: attempt to remap topics for cartographer

File: src/vineyard_mower_description/urdf/vineyard_mower.urdf.xacro (robot description, xacro)
@@ -186,4 +186,17 @@
     <origin xyz="0 0 ${sensor_height + 0.025}" rpy="0 0 0"/>
   </joint>
+  <!-- Create a frame for Cartographer compatibility -->
+  <link name="lidar">
+    <inertial>
+      <origin xyz="0 0 0" rpy="0 0 0"/>
+      <mass value="0.001"/>
+      <inertia ixx="0.0001" ixy="0" ixz="0" iyy="0.0001" iyz="0" izz="0.0001"/>
+    </inertial>
+  </link>
+  <joint name="lidar_alias_joint" type="fixed">
+    <parent link="lidar_link"/>
+    <child link="lidar"/>
+    <origin xyz="0 0 0" rpy="0 0 0"/>
+  </joint>
   <!-- Front camera (Intel RealSense) -->
   <link name="front_camera_link">
@@ -310,5 +323,5 @@
     <!-- <sensor name="gpu_lidar" type="gpu_lidar">
      -->
-      <sensor name="lidar" type="gpu_lidar">
+      <sensor name="lidar_link" type="gpu_lidar">
       <pose>0 0 0 0 0 0</pose>
       <topic>scan</topic>

Commit message: fix: weel width, location

File: src/vineyard_mower_description/urdf/vineyard_mower.urdf.xacro (robot description, xacro)
@@ -10,5 +10,5 @@
   <!-- Wheel properties -->
   <xacro:property name="wheel_radius" value="0.15"/>
-  <xacro:property name="wheel_width" value="0.3"/>
+  <xacro:property name="wheel_width" value="0.1"/>
   <xacro:property name="track_width" value="1.4"/>
   <!-- Sensor properties -->
@@ -83,5 +83,5 @@
   <link name="left_wheel">
     <visual>
-      <origin xyz="0 0 0" rpy="${PI/2} 0 0"/>
+      <origin xyz="-0.1 0 0" rpy="${PI/2} 0 0"/>
       <geometry>
         <cylinder radius="${wheel_radius}" length="${wheel_width}"/>
@@ -90,5 +90,5 @@
     </visual>
     <collision>
-      <origin xyz="0 0 0" rpy="${PI/2} 0 0"/>
+      <origin xyz="-0.1 0 0" rpy="${PI/2} 0 0"/>
       <geometry>
         <cylinder radius="${wheel_radius}" length="${wheel_width}"/>
@@ -96,5 +96,5 @@
     </collision>
     <inertial>
-      <origin xyz="0 0 0" rpy="${PI/2} 0 0"/>
+      <origin xyz="-0.1 0 0" rpy="${PI/2} 0 0"/>
       <mass value="5.0"/>
       <inertia ixx="0.1125" ixy="0" ixz="0" iyy="0.1125" iyz="0" izz="0.1125"/>
@@ -110,5 +110,5 @@
   <link name="right_wheel">
     <visual>
-      <origin xyz="0 0 0" rpy="${PI/2} 0 0"/>
+      <origin xyz="0.1 0 0" rpy="${PI/2} 0 0"/>
       <geometry>
         <cylinder radius="${wheel_radius}" length="${wheel_width}"/>
@@ -117,5 +117,5 @@
     </visual>
     <collision>
-      <origin xyz="0 0 0" rpy="${PI/2} 0 0"/>
+      <origin xyz="0.1 0 0" rpy="${PI/2} 0 0"/>
       <geometry>
         <cylinder radius="${wheel_radius}" length="${wheel_width}"/>
@@ -123,5 +123,5 @@
     </collision>
     <inertial>
-      <origin xyz="0 0 0" rpy="${PI/2} 0 0"/>
+      <origin xyz="0.1 0 0" rpy="${PI/2} 0 0"/>
       <mass value="5.0"/>
       <inertia ixx="0.1125" ixy="0" ixz="0" iyy="0.1125" iyz="0" izz="0.1125"/>

Commit message: fix: base footprint

File: src/vineyard_mower_description/urdf/vineyard_mower.urdf.xacro (robot description, xacro)
@@ -33,4 +33,17 @@
     <color rgba="0.0 0.0 0.8 1.0"/>
   </material>
+  <!-- Base Footprint (for ground reference) -->
+  <link name="base_footprint">
+    <inertial>
+      <mass value="0.0001"/>
+      <origin xyz="0 0 0"/>
+      <inertia ixx="0.0001" ixy="0.0" ixz="0.0" iyy="0.0001" iyz="0.0" izz="0.0001"/>
+    </inertial>
+  </link>
+  <joint name="base_footprint_joint" type="fixed">
+    <parent link="base_footprint"/>
+    <child link="base_link"/>
+    <origin xyz="0 0 ${wheel_radius}" rpy="0 0 0"/>
+  </joint>
   <!-- Base Link -->
   <link name="base_link">
@@ -83,5 +96,5 @@
   <link name="left_wheel">
     <visual>
-      <origin xyz="-0.1 0 0" rpy="${PI/2} 0 0"/>
+      <origin xyz="0 0 0" rpy="${PI/2} 0 0"/>
       <geometry>
         <cylinder radius="${wheel_radius}" length="${wheel_width}"/>
@@ -90,5 +103,5 @@
     </visual>
     <collision>
-      <origin xyz="-0.1 0 0" rpy="${PI/2} 0 0"/>
+      <origin xyz="0 0 0" rpy="${PI/2} 0 0"/>
       <geometry>
         <cylinder radius="${wheel_radius}" length="${wheel_width}"/>
@@ -96,5 +109,5 @@
     </collision>
     <inertial>
-      <origin xyz="-0.1 0 0" rpy="${PI/2} 0 0"/>
+      <origin xyz="0 0 0" rpy="${PI/2} 0 0"/>
       <mass value="5.0"/>
       <inertia ixx="0.1125" ixy="0" ixz="0" iyy="0.1125" iyz="0" izz="0.1125"/>
@@ -104,5 +117,5 @@
     <parent link="base_link"/>
     <child link="left_wheel"/>
-    <origin xyz="0 ${track_width/2} ${wheel_radius}" rpy="0 0 0"/>
+    <origin xyz="0 ${track_width/2} 0" rpy="0 0 0"/>
     <axis xyz="0 1 0"/>
   </joint>
@@ -110,5 +123,5 @@
   <link name="right_wheel">
     <visual>
-      <origin xyz="0.1 0 0" rpy="${PI/2} 0 0"/>
+      <origin xyz="0 0 0" rpy="${PI/2} 0 0"/>
       <geometry>
         <cylinder radius="${wheel_radius}" length="${wheel_width}"/>
@@ -117,5 +130,5 @@
     </visual>
     <collision>
-      <origin xyz="0.1 0 0" rpy="${PI/2} 0 0"/>
+      <origin xyz="0 0 0" rpy="${PI/2} 0 0"/>
       <geometry>
         <cylinder radius="${wheel_radius}" length="${wheel_width}"/>
@@ -123,5 +136,5 @@
     </collision>
     <inertial>
-      <origin xyz="0.1 0 0" rpy="${PI/2} 0 0"/>
+      <origin xyz="0 0 0" rpy="${PI/2} 0 0"/>
       <mass value="5.0"/>
       <inertia ixx="0.1125" ixy="0" ixz="0" iyy="0.1125" iyz="0" izz="0.1125"/>
@@ -131,5 +144,5 @@
     <parent link="base_link"/>
     <child link="right_wheel"/>
-    <origin xyz="0 ${-track_width/2} ${wheel_radius}" rpy="0 0 0"/>
+    <origin xyz="0 ${-track_width/2} 0" rpy="0 0 0"/>
     <axis xyz="0 1 0"/>
   </joint>

Commit message: fix: wheel position

File: src/vineyard_mower_description/urdf/vineyard_mower.urdf.xacro (robot description, xacro)
@@ -117,5 +117,5 @@
     <parent link="base_link"/>
     <child link="left_wheel"/>
-    <origin xyz="0 ${track_width/2} 0" rpy="0 0 0"/>
+    <origin xyz="0 ${track_width/2+0.1} 0.1" rpy="0 0 0"/>
     <axis xyz="0 1 0"/>
   </joint>
@@ -144,5 +144,5 @@
     <parent link="base_link"/>
     <child link="right_wheel"/>
-    <origin xyz="0 ${-track_width/2} 0" rpy="0 0 0"/>
+    <origin xyz="0 ${-track_width/2-0.1} 0.1" rpy="0 0 0"/>
     <axis xyz="0 1 0"/>
   </joint>

Commit message: feat: add front, rear caster joint

File: src/vineyard_mower_description/urdf/vineyard_mower.urdf.xacro (robot description, xacro)
@@ -34,15 +34,61 @@
   </material>
   <!-- Base Footprint (for ground reference) -->
-  <link name="base_footprint">
-    <inertial>
-      <mass value="0.0001"/>
-      <origin xyz="0 0 0"/>
-      <inertia ixx="0.0001" ixy="0.0" ixz="0.0" iyy="0.0001" iyz="0.0" izz="0.0001"/>
-    </inertial>
-  </link>
+  <link name="base_footprint"/>
   <joint name="base_footprint_joint" type="fixed">
     <parent link="base_footprint"/>
     <child link="base_link"/>
     <origin xyz="0 0 ${wheel_radius}" rpy="0 0 0"/>
+  </joint>
+  <!-- Front Caster Sphere -->
+  <link name="front_caster">
+    <visual>
+      <origin xyz="0 0 0" rpy="0 0 0"/>
+      <geometry>
+        <sphere radius="0.05"/>
+      </geometry>
+      <material name="grey"/>
+    </visual>
+    <collision>
+      <origin xyz="0 0 0" rpy="0 0 0"/>
+      <geometry>
+        <sphere radius="0.05"/>
+      </geometry>
+    </collision>
+    <inertial>
+      <mass value="0.5"/>
+      <origin xyz="0 0 0"/>
+      <inertia ixx="0.0005" ixy="0.0" ixz="0.0" iyy="0.0005" iyz="0.0" izz="0.0005"/>
+    </inertial>
+  </link>
+  <joint name="front_caster_joint" type="fixed">
+    <parent link="base_link"/>
+    <child link="front_caster"/>
+    <origin xyz="${base_length/2 + 0.05} 0 0" rpy="0 0 0"/>
+  </joint>
+  <!-- Rear Caster Sphere -->
+  <link name="rear_caster">
+    <visual>
+      <origin xyz="0 0 0" rpy="0 0 0"/>
+      <geometry>
+        <sphere radius="0.05"/>
+      </geometry>
+      <material name="grey"/>
+    </visual>
+    <collision>
+      <origin xyz="0 0 0" rpy="0 0 0"/>
+      <geometry>
+        <sphere radius="0.05"/>
+      </geometry>
+    </collision>
+    <inertial>
+      <mass value="0.5"/>
+      <origin xyz="0 0 0"/>
+      <inertia ixx="0.0005" ixy="0.0" ixz="0.0" iyy="0.0005" iyz="0.0" izz="0.0005"/>
+    </inertial>
+  </link>
+  <joint name="rear_caster_joint" type="fixed">
+    <parent link="base_link"/>
+    <child link="rear_caster"/>
+    <origin xyz="${-base_length/2 - 0.05} 0 0" rpy="0 0 0"/>
   </joint>
   <!-- Base Link -->
@@ -290,4 +336,20 @@
     <maxVel>1.0</maxVel>
     <fdir1>1 0 0</fdir1>
+  </gazebo>
+  <gazebo reference="front_caster">
+    <material>Gazebo/Grey</material>
+    <mu1>0.0</mu1>
+    <mu2>0.0</mu2>
+    <kp>1000000.0</kp>
+    <kd>100.0</kd>
+    <minDepth>0.001</minDepth>
+  </gazebo>
+  <gazebo reference="rear_caster">
+    <material>Gazebo/Grey</material>
+    <mu1>0.0</mu1>
+    <mu2>0.0</mu2>
+    <kp>1000000.0</kp>
+    <kd>100.0</kd>
+    <minDepth>0.001</minDepth>
   </gazebo>
   <gazebo reference="lidar_link">
